File: Hardware/Qwiic_FM_Transceiver_Si4721.sch (EAGLE design)
At the start: 37 parts, among them J1 AUDIO_JACK_3.5MM_SMD, J2 AUDIO_JACK_3.5MM_SMD, J4 QWIIC_RIGHT_ANGLE, J5 QWIIC_RIGHT_ANGLE, U3 TPA6111, Y1 32.768kHz

Commit message: x01
x01
Parts:
- removed R9: 10k, SparkFun-Resistors:10KOHM-0603-1/10W-1%
- added FD1, FD2: FIDUCIAL0.2MM, SparkFun-Aesthetics:FIDUCIAL0.2MM
- added H1, H2, H3, H4: STAND-OFF, SparkFun-Hardware:STAND-OFF
- added R10: 100k, SparkFun-Resistors:100KOHM-0603-1/10W-1%
- added U$18: SPARKX-LOGO4, SparkX:SPARKX-LOGO4
- C12: device SparkFun-Capacitors:22NF/22,000PF-50V-10%(0603) -> SparkFun-Capacitors:22NF/22,000PF-0603-50V-10%
- C6, C9: device SparkFun-Capacitors:0.1UF-25V(+80/-20%)(0603) -> SparkFun-Capacitors:0.1UF-0603-25V-(+80/-20%)
- C7, C8: device SparkFun-Capacitors:47UF-TANT -> SparkFun-Capacitors:47UF-POLAR-EIA3528-10V-10%
- JP1: value JUMPER-SMT_3_2-NC_TRACE_NO-SILK -> JUMPER-SMT_3_2-NC_TRACE_SILK; device SparkFun-Jumpers:JUMPER-SMT_3_2-NC_TRACE_NO-SILK -> SparkFun-Jumpers:JUMPER-SMT_3_2-NC_TRACE_SILK
- JP2: value JUMPER-SMT_3_2-NC_TRACE_NO-SILK -> JUMPER-SMT_2_NC_TRACE_SILK; device SparkFun-Jumpers:JUMPER-SMT_3_2-NC_TRACE_NO-SILK -> SparkFun-Jumpers:JUMPER-SMT_2_NC_TRACE_SILK
- L2: value Ferrite 2.5k -> FERITE 2.5k; device SparkFun-Passives:INDUCTOR0603 -> SparkFun-Coils:FERRITE_BEAD-0603
- L3: value Ferrite 2.5k -> FERITE 2.5K; device SparkFun-Passives:INDUCTOR0603 -> SparkFun-Coils:FERRITE_BEAD-0603
- R4, R5, R6, R7: device SparkFun-Resistors:20KOHM1/10W1%(0603) -> SparkFun-Resistors:20KOHM-0603-1/10W-5%
- U3: value TPA6111 -> TPA6111A2DR; device SparkFun-AnalogIC:TPA6111SMD-T -> SparkFun-IC-Amplifiers:TPA6111SMD-T
- renumbered U$1 to U1
Connections:
- removed net N$23: JP2.2, R9.1
- removed net RFGND: J3.2, U1.RFGND
- net 3.3V: now also R10.2; no longer JP2.3
- net ADDR: now also JP2.1, R10.1; no longer R9.2
- net GND: now also J3.1, JP2.2, U1.RFGND; no longer JP2.1
- net TXO: now also J3.2; no longer J3.1
Other:
- note added: "TODO: Note about antenna length/material"
- note added: "address is determined by !SEN LOW addr = 0010001 (0x11) HIGH addr = 1100011 (0x63)"
- moved on the sheet: J3, JP1, R2, R3

Commit message: x02 hardware order
Parts:
- added C13: 2.2uF, SparkFun-Capacitors:2.2UF-0603-10V-20%
Connections:
- net GND: now also C13.2
- net N$1: now also C13.1
Other:
- note added: "!RST needs to come up after VDD to boot into I2C mode. 2.2uF is chosen because we have it in stock. Should provide about 20ms from power applied to !RST > 0.7*VDD"
- moved on the sheet: R1
Changed lines of the file:
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@@
 <?xml version="1.0" encoding="utf-8"?>
 <!DOCTYPE eagle SYSTEM "eagle.dtd">
-<eagle version="9.5.0">
+<eagle version="9.5.1">
 <drawing>
 <settings>
@@
 <layer number="1" name="Top" color="4" fill="1" visible="no" active="no"/>
 <layer number="2" name="Route2" color="1" fill="3" visible="no" active="no"/>
+<layer number="3" name="Route3" color="4" fill="3" visible="no" active="no"/>
+<layer number="4" name="Route4" color="1" fill="4" visible="no" active="no"/>
+<layer number="5" name="Route5" color="4" fill="4" visible="no" active="no"/>
+<layer number="6" name="Route6" color="1" fill="8" visible="no" active="no"/>
+<layer number="7" name="Route7" color="4" fill="8" visible="no" active="no"/>
+<layer number="8" name="Route8" color="1" fill="2" visible="no" active="no"/>
+<layer number="9" name="Route9" color="4" fill="2" visible="no" active="no"/>
+<layer number="10" name="Route10" color="1" fill="7" visible="no" active="no"/>
+<layer number="11" name="Route11" color="4" fill="7" visible="no" active="no"/>
+<layer number="12" name="Route12" color="1" fill="5" visible="no" active="no"/>
+<layer number="13" name="Route13" color="4" fill="5" visible="no" active="no"/>
+<layer number="14" name="Route14" color="1" fill="6" visible="no" active="no"/>
 <layer number="15" name="Route15" color="4" fill="6" visible="no" active="no"/>
 <layer number="16" name="Bottom" color="1" fill="1" visible="no" active="no"/>
@@
 <part name="JP2" library="SparkFun-Jumpers" deviceset="JUMPER-SMT_2_NC_TRACE" device="_SILK" value=""/>
 <part name="R10" library="SparkFun-Resistors" deviceset="100KOHM" device="-0603-1/10W-1%" value="100k"/>
+<part name="C13" library="SparkFun-Capacitors" deviceset="2.2UF" device="-0603-10V-20%" value="2.2uF"/>
+<part name="GND15" library="SparkFun-PowerSymbols" deviceset="GND" device=""/>
 </parts>
 <sheets>
@@
 HIGH addr = 1100011 (0x63)</text>
 <text x="177.8" y="181.864" size="1.27" layer="94">TODO: Note about antenna length/material</text>
+<text x="2.54" y="177.8" size="1.27" layer="94">!RST needs to come up after VDD to boot into I2C mode.
+2.2uF is chosen because we have it in stock.
+Should provide about 20ms from power applied to !RST &gt; 0.7*VDD</text>
 </plain>
 <instances>
@@
 <attribute name="VALUE" x="83.82" y="155.194" size="1.778" layer="96" align="bottom-center"/>
 </instance>
-<instance part="R1" gate="G$1" x="25.4" y="162.56" smashed="yes" rot="R270">
-<attribute name="NAME" x="26.924" y="167.64" size="1.778" layer="95" font="vector" rot="R270" align="bottom-center"/>
-<attribute name="VALUE" x="28.956" y="160.02" size="1.778" layer="96" font="vector" rot="R270" align="top-center"/>
-</instance>
-<instance part="SUPPLY2" gate="G$1" x="25.4" y="170.18" smashed="yes">
-<attribute name="VALUE" x="25.4" y="172.974" size="1.778" layer="96" align="bottom-center"/>
+<instance part="R1" gate="G$1" x="22.86" y="162.56" smashed="yes" rot="R270">
+<attribute name="NAME" x="24.384" y="167.64" size="1.778" layer="95" font="vector" rot="R270" align="bottom-center"/>
+<attribute name="VALUE" x="26.416" y="160.02" size="1.778" layer="96" font="vector" rot="R270" align="top-center"/>
+</instance>
+<instance part="SUPPLY2" gate="G$1" x="22.86" y="170.18" smashed="yes">
+<attribute name="VALUE" x="22.86" y="172.974" size="1.778" layer="96" align="bottom-center"/>
 </instance>
 <instance part="J1" gate="G$1" x="223.52" y="73.66" smashed="yes" rot="MR0">
@@
 <attribute name="NAME" x="147.32" y="174.244" size="1.778" layer="95" font="vector" align="bottom-center"/>
 <attribute name="VALUE" x="147.32" y="171.196" size="1.778" layer="96" font="vector" align="top-center"/>
+</instance>
+<instance part="C13" gate="G$1" x="22.86" y="147.32" smashed="yes">
+<attribute name="NAME" x="24.384" y="150.241" size="1.778" layer="95" font="vector"/>
+<attribute name="VALUE" x="24.384" y="145.161" size="1.778" layer="96" font="vector"/>
+</instance>
+<instance part="GND15" gate="1" x="22.86" y="139.7" smashed="yes">
+<attribute name="VALUE" x="22.86" y="139.446" size="1.778" layer="96" align="top-center"/>
 </instance>
 </instances>
@@
 <wire x1="139.7" y1="157.48" x2="139.7" y2="160.02" width="0.1524" layer="91"/>
 </segment>
+<segment>
+<pinref part="C13" gate="G$1" pin="2"/>
+<wire x1="22.86" y1="144.78" x2="22.86" y2="142.24" width="0.1524" layer="91"/>
+<pinref part="GND15" gate="1" pin="GND"/>
+</segment>
 </net>
 <net name="LIN" class="0">
@@
 <segment>
 <pinref part="R1" gate="G$1" pin="1"/>
-<wire x1="25.4" y1="167.64" x2="25.4" y2="170.18" width="0.1524" layer="91"/>
+<wire x1="22.86" y1="167.64" x2="22.86" y2="170.18" width="0.1524" layer="91"/>
 <pinref part="SUPPLY2" gate="G$1" pin="3.3V"/>
 </segment>
@@
 <pinref part="R1" gate="G$1" pin="2"/>
 <pinref part="U1" gate="G$1" pin="!RST"/>
-<wire x1="25.4" y1="157.48" x2="25.4" y2="154.94" width="0.1524" layer="91"/>
-<wire x1="25.4" y1="154.94" x2="40.64" y2="154.94" width="0.1524" layer="91"/>
-</segment>
-</net>
+<wire x1="22.86" y1="157.48" x2="22.86" y2="154.94" width="0.1524" layer="91"/>
+<wire x1="22.86" y1="154.94" x2="40.64" y2="154.94" width="0.1524" layer="91"/>
+<wire x1="22.86" y1="154.94" x2="22.86" y2="152.4" width="0.1524" layer="91"/>
+<junction x="22.86" y="154.94"/>
+<pinref part="C13" gate="G$1" pin="1"/>
+</segment>
+</net>
